File: hardware/miniadapter/board_connectionpcb/connectionpcb.kicad_sch (KiCad schematic)
At the start: 11 parts

Commit message: new layout
Parts:
- removed TP101, TP102, TP103, TP104, TP105, TP106, TP107, TP108, TP109, TP110: TestPoint, TestPoint:TestPoint_Pad_1.0x1.0mm, symbol Connector:TestPoint
- added J101: Conn_01x04, minipcb:minipcb_alt_boardedge, symbol Connector_Generic:Conn_01x04
- added J102: Conn_02x03_Odd_Even, minipcb:ESP8685-WROOM-07, symbol Connector_Generic:Conn_02x03_Odd_Even
Connections:
- net ANT: now also J102.1 (Pin_1); no longer AE101.1 (A)
- net GND: now also J101.1 (Pin_1), J102.2 (Pin_2); no longer AE101.2 (Shield)
- new net +3V3: J101.4 (Pin_4), J102.6 (Pin_6)
- new net IO10: J102.5 (Pin_5)
- new net IO4: J101.3 (Pin_3), J102.4 (Pin_4)
- new net IO5: J101.2 (Pin_2), J102.3 (Pin_3)

Commit message: layout changes and panel generation
Parts:
- AE101: OC_JLC (none) -> C2925416
Changed lines of the file:
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@@
+			)
+		)
+		(property "OC_JLC" "C2925416"
+			(at 172.72 54.61 0)
+			(effects
+				(font
+					(size 1.27 1.27)
+				)
+				(hide yes)
 			)
 		)
